File: KiPad.kicad_sch (KiCad schematic)
At the start: 66 parts, among them J1 USB_C_Receptacle_USB2.0, SW1 SW_SPST_LED, SW10 SW_SPST, SW11 SW_SPST, SW12 SW_SPST, SW13 SW_SPST, SW14 SW_SPST, SW15 SW_SPST, SW16 SW_SPST, SW17 SW_SPST, SW18 SW_SPST, SW19 SW_SPST, SW2 SW_SPST_LED, SW20 SW_SPST, SW21 SW_SPST, SW3 SW_SPST_LED, SW4 SW_SPST_LED, SW5 SW_SPST, SW6 SW_SPST, SW7 SW_SPST, SW8 SW_SPST, SW9 SW_SPST, U1 ATmega32U4RC-A, Y1 16MHz

Commit message: v2
Parts:
- removed C1: 1u, Capacitor_SMD:C_0805_2012Metric, symbol Device:C
- removed C3, C4: 22p, Capacitor_SMD:C_0805_2012Metric, symbol Device:C_Small
- removed F1: 500mA, Fuse:Fuse_1206_3216Metric, symbol Device:Polyfuse
- removed J1: USB_C_Receptacle_USB2.0, Connector_USB:USB_C_Receptacle_GCT_USB4105-xx-A_16P_TopMnt_Horizontal, symbol Connector:USB_C_Receptacle_USB2.0_14P
- removed R1, R2: 22, Resistor_SMD:R_0805_2012Metric, symbol Device:R
- removed R10, R11: 10k, Resistor_SMD:R_0805_2012Metric, symbol Device:R
- removed R3, R4: 5.1k, Resistor_SMD:R_0805_2012Metric, symbol Device:R
- removed SW_HWB1, SW_RST1: SW_Push, Button_Switch_SMD:SW_SPST_TL3342, symbol Switch:SW_Push
- removed U1: ATmega32U4RC-A, Package_QFP:TQFP-44_10x10mm_P0.8mm, symbol MCU_Microchip_ATmega:ATmega32U4RC-A
- removed Y1: 16MHz, Crystal:Crystal_SMD_3225-4Pin_3.2x2.5mm, symbol Device:Crystal_GND24
- added J1, J2: Conn_02x08_Counter_Clockwise, Connector_PinSocket_2.54mm:PinSocket_2x08_P2.54mm_Vertical, symbol Connector_Generic:Conn_02x08_Odd_Even
- A1: footprint Custom:KB2040_SMD -> Custom:KB2040_THT; DIGIKEY (none) -> 1528-5302-ND
- SW1, SW2, SW3, SW4: footprint Custom:MX-Solderable-1U-0805-LED -> Custom:MX-Hotswap-1U-0805-LED
- SW10, SW11, SW13, SW14, SW15, SW16, SW17, SW18, SW21, SW5, SW6, SW7, SW8, SW9: footprint MX_Solderable:MX-Solderable-1U -> MX_Hotswap:MX-Hotswap-1U
- SW12, SW19: footprint MX_Solderable:MX-Solderable-2U-Vertical -> MX_Hotswap:MX-Hotswap-2U-Vertical-ReversedStabilizers
- SW20: footprint MX_Solderable:MX-Solderable-2U -> MX_Hotswap:MX-Hotswap-2U
Connections:
- net C0: now also J1.8 (Pin_8); no longer A1.2 (D0)
- net C1: now also J1.6 (Pin_6); no longer A1.3 (D1)
- net C2: now also J1.4 (Pin_4); no longer A1.6 (D2)
- net C3: now also J1.2 (Pin_2); no longer A1.7 (D3)
- net GND: now also J1.5 (Pin_5); no longer A1.24 (GND), A1.4 (GND), A1.5 (GND)
- net LED_A: now also J1.13 (Pin_13); no longer A1.18 (A0)
- net LED_B: now also J1.11 (Pin_11); no longer A1.19 (A1)
- net LED_C: now also J1.9 (Pin_9); no longer A1.20 (A2)
- net LED_D: now also J1.7 (Pin_7); no longer A1.21 (A3)
- net R0: now also J1.1 (Pin_1); no longer A1.8 (D4)
- net R1: now also J1.15 (Pin_15); no longer A1.9 (D5)
- net R2: now also J1.16 (Pin_16); no longer A1.10 (D6)
- net R3: now also J1.14 (Pin_14); no longer A1.11 (D7)
- net R4: now also J1.12 (Pin_12); no longer A1.12 (D8)
- net R5: now also J1.10 (Pin_10); no longer A1.13 (D9)
- net MCU_R1: now reaches A1.14 (D10)
- net MCU_R1: now also J2.15 (Pin_15)
- net +5V renamed +3V3
- net +3V3: now also J1.3 (Pin_3); no longer A1.22 (3V3)
- new net MCU_C0: A1.9 (D5), J2.8 (Pin_8)
- new net MCU_C1: A1.10 (D6), J2.6 (Pin_6)
- new net MCU_C2: A1.11 (D7), J2.4 (Pin_4)
- new net MCU_C3: A1.12 (D8), J2.2 (Pin_2)
- new net MCU_GND: A1.24 (GND), A1.4 (GND), A1.5 (GND), J2.5 (Pin_5)
- new net MCU_LED_A: A1.18 (A0), J2.13 (Pin_13)
- new net MCU_LED_B: A1.19 (A1), J2.11 (Pin_11)
- new net MCU_LED_C: A1.20 (A2), J2.9 (Pin_9)
- new net MCU_LED_D: A1.21 (A3), J2.7 (Pin_7)
- new net MCU_R0: A1.13 (D9), J2.1 (Pin_1)
- new net MCU_R2: A1.3 (D1), J2.16 (Pin_16)
- new net MCU_R3: A1.6 (D2), J2.14 (Pin_14)
- new net MCU_R4: A1.7 (D3), J2.12 (Pin_12)
- new net MCU_R5: A1.8 (D4), J2.10 (Pin_10)
- new net MCU_VCC: A1.22 (3V3), J2.3 (Pin_3)
- no-connect marks 20 -> 8
Other:
- note removed: "Crystal"
- note removed: "Reset & Flash"
- moved on the sheet: A1

Commit message: v3
Parts:
- removed A1: Adafruit Key Boar KB2040, Custom:KB2040_THT, symbol Custom:Adafruit_KB2040
- removed J1, J2: Conn_02x08_Counter_Clockwise, Connector_PinSocket_2.54mm:PinSocket_2x08_P2.54mm_Vertical, symbol Connector_Generic:Conn_02x08_Odd_Even
- removed R6, R7, R8, R9: 470, Resistor_SMD:R_0805_2012Metric, symbol Device:R
- added C1, C3: 22p, Capacitor_SMD:C_0402_1005Metric, symbol Device:C
- added J1: USB_C_Receptacle_USB2.0_14P, Connector_USB:USB_C_Receptacle_GCT_USB4105-xx-A_16P_TopMnt_Horizontal, symbol Connector:USB_C_Receptacle_USB2.0_14P
- added LED1, LED10, LED11, LED12, LED13, LED14, LED15, LED16, LED17, LED18, LED19, LED2, LED20, LED21, LED3, LED4, LED5, LED6, LED7, LED8, LED9: SK6812MINI, Custom:LED_SK6812MINI-E_PLCC4_3.2x2.8mm_P1.75mm, symbol Custom:SK6812MINI-E
- added R1: 10k, Resistor_SMD:R_0402_1005Metric, symbol Device:R
- added R2, R3: 5.1k, Resistor_SMD:R_0402_1005Metric, symbol Device:R
- added R4, R5: 22, Resistor_SMD:R_0402_1005Metric, symbol Device:R
- added SW22: RESET, Resistor_SMD:R_0603_1608Metric, symbol Switch:SW_Push
- added U2: ATmega32U2-M, Package_DFN_QFN:QFN-32-1EP_5x5mm_P0.5mm_EP3.1x3.1mm, symbol MCU_Microchip_ATmega:ATmega32U2-M
- added Y1: 16MHz, Crystal:Crystal_SMD_3225-4Pin_3.2x2.5mm, symbol Device:Crystal_GND24
- C6: value 0.1u -> 1u; footprint Capacitor_SMD:C_0805_2012Metric -> Capacitor_SMD:C_0603_1608Metric; DIGIKEY 478-KGM21NR71H104KTTR-ND -> 311-1446-1-ND
- SW1: value SW_SPST_LED -> SW_A; footprint Custom:MX-Hotswap-1U-0805-LED -> MX_Hotswap:MX-Hotswap-1U; symbol Switch:SW_SPST_LED -> Switch:SW_SPST; DIGIKEY 1497-1450-1-ND -> (none)
- SW10: value SW_SPST -> SW_8
- SW11: value SW_SPST -> SW_9
- SW12: value SW_SPST -> SW_ADD
- SW13: value SW_SPST -> SW_4
- SW14: value SW_SPST -> SW_5
- SW15: value SW_SPST -> SW_6
- SW16: value SW_SPST -> SW_1
- SW17: value SW_SPST -> SW_2
- SW18: value SW_SPST -> SW_3
- SW19: value SW_SPST -> SW_ENTER
- SW2: value SW_SPST_LED -> SW_B; footprint Custom:MX-Hotswap-1U-0805-LED -> MX_Hotswap:MX-Hotswap-1U; symbol Switch:SW_SPST_LED -> Switch:SW_SPST; DIGIKEY 1497-1450-1-ND -> (none)
- SW20: value SW_SPST -> SW_0
- SW21: value SW_SPST -> SW_DOT
- SW3: value SW_SPST_LED -> SW_C; footprint Custom:MX-Hotswap-1U-0805-LED -> MX_Hotswap:MX-Hotswap-1U; symbol Switch:SW_SPST_LED -> Switch:SW_SPST; DIGIKEY 1497-1450-1-ND -> (none)
- SW4: value SW_SPST_LED -> SW_D; footprint Custom:MX-Hotswap-1U-0805-LED -> MX_Hotswap:MX-Hotswap-1U; symbol Switch:SW_SPST_LED -> Switch:SW_SPST; DIGIKEY 1497-1450-1-ND -> (none)
- SW5: value SW_SPST -> SW_NL
- SW6: value SW_SPST -> SW_DIV
- SW7: value SW_SPST -> SW_MUL
- SW8: value SW_SPST -> SW_SUB
- SW9: value SW_SPST -> SW_7
- renumbered D18 to D1, D6 to D10, D7 to D11, D8 to D12, D9 to D13, D10 to D14, D11 to D15, D12 to D16, D13 to D17, D14 to D18, D15 to D19, D19 to D2, D16 to D20, D17 to D21, D20 to D3, D21 to D4, D1 to D5, D2 to D6, D3 to D7, D4 to D8, D5 to D9
Connections:
- net C0: now also U2.9 (PD3)
- net C1: now also U2.23 (PC6)
- net C2: now also U2.21 (PB7)
- net C3: now also U2.20 (PB6)
- net GND: now also C1.1, C3.2, J1.A1 (GND), J1.A12 (GND), J1.B1 (GND), J1.B12 (GND), J1.S1 (SHIELD), LED1.3 (VSS), LED10.3 (VSS), LED11.3 (VSS), LED12.3 (VSS), LED13.3 (VSS), LED14.3 (VSS), LED15.3 (VSS), LED16.3 (VSS), LED17.3 (VSS), LED18.3 (VSS), LED19.3 (VSS), LED2.3 (VSS), LED20.3 (VSS), LED21.3 (VSS), LED3.3 (VSS), LED4.3 (VSS), LED5.3 (VSS), LED6.3 (VSS), LED7.3 (VSS), LED8.3 (VSS), LED9.3 (VSS), R2.2, R3.2, SW22.2, U2.28 (UGND), U2.3 (GND), U2.33 (GND), Y1.2, Y1.4
- net R0: now also U2.14 (PB0)
- net R1: now also U2.16 (PB2)
- net R2: now also U2.25 (PC5)
- net R3: now also U2.22 (PC7)
- net R4: now also U2.11 (PD5)
- net R5: now also U2.10 (PD4)
- removed net +3V3: C2.1, C5.1, C6.1, C7.1, SW1.4 (A), SW2.4 (A), SW3.4 (A), SW4.4 (A)
- new net: LED4.2 (DOUT), LED5.4 (DIN)
- new net: LED3.2 (DOUT), LED4.4 (DIN)
- new net: C6.1, U2.27 (UCAP)
- new net: LED14.2 (DOUT), LED15.4 (DIN)
- new net: LED13.2 (DOUT), LED14.4 (DIN)
- new net: LED17.2 (DOUT), LED18.4 (DIN)
- new net: LED16.2 (DOUT), LED17.4 (DIN)
- new net: LED6.2 (DOUT), LED7.4 (DIN)
- new net: LED5.2 (DOUT), LED6.4 (DIN)
- new net: LED2.2 (DOUT), LED3.4 (DIN)
- new net: LED1.2 (DOUT), LED2.4 (DIN)
- new net: R1.2, SW22.1, U2.24 (PC1/~{RESET})
- new net: LED10.2 (DOUT), LED11.4 (DIN)
- new net: LED10.4 (DIN), LED9.2 (DOUT)
- new net: C3.1, U2.2 (PC0/XTAL2), Y1.3
- new net: J1.A5 (CC1), R3.1
- new net: J1.A6 (D+), J1.B6 (D+), R5.1
- new net: J1.A7 (D-), J1.B7 (D-), R4.1
- new net: J1.B5 (CC2), R2.1
- new net: C1.2, U2.1 (XTAL1), Y1.1
- new net: LED15.2 (DOUT), LED16.4 (DIN)
- new net: LED12.2 (DOUT), LED13.4 (DIN)
- new net: LED11.2 (DOUT), LED12.4 (DIN)
- new net: LED8.2 (DOUT), LED9.4 (DIN)
- new net: LED20.2 (DOUT), LED21.4 (DIN)
- new net: LED19.2 (DOUT), LED20.4 (DIN)
- new net: LED7.2 (DOUT), LED8.4 (DIN)
- new net: LED18.2 (DOUT), LED19.4 (DIN)
- new net +5V: C2.1, C5.1, C7.1, J1.A4 (VBUS), J1.A9 (VBUS), J1.B4 (VBUS), J1.B9 (VBUS), LED1.1 (VDD), LED10.1 (VDD), LED11.1 (VDD), LED12.1 (VDD), LED13.1 (VDD), LED14.1 (VDD), LED15.1 (VDD), LED16.1 (VDD), LED17.1 (VDD), LED18.1 (VDD), LED19.1 (VDD), LED2.1 (VDD), LED20.1 (VDD), LED21.1 (VDD), LED3.1 (VDD), LED4.1 (VDD), LED5.1 (VDD), LED6.1 (VDD), LED7.1 (VDD), LED8.1 (VDD), LED9.1 (VDD), R1.1, U2.31 (UVCC), U2.32 (AVCC), U2.4 (VCC)
- new net LED_DATA: LED1.4 (DIN), U2.15 (PB1)
- new net USB_DN: R4.2, U2.30 (D-)
- new net USB_DP: R5.2, U2.29 (D+)
- no-connect marks 8 -> 1
Other:
- note added: "LEDs"
- moved on the sheet: C6, C7, D1, D2, D3, D4

Commit message: v3.1
Flip around stabs so the shaft is on the outside.
Fix LED footprint and reroute.
Parts:
- J1: symbol Connector:USB_C_Receptacle_USB2.0_14P -> Connector:USB_C_Receptacle_USB2.0_16P
- SW12, SW19: footprint MX_Hotswap:MX-Hotswap-2U-Vertical-ReversedStabilizers -> MX_Hotswap:MX-Hotswap-2U-Vertical
- SW20: footprint MX_Hotswap:MX-Hotswap-2U -> MX_Hotswap:MX-Hotswap-2U-ReversedStabilizers
- SW22: footprint Resistor_SMD:R_0603_1608Metric -> Resistor_SMD:R_0402_1005Metric_Pad0.72x0.64mm_HandSolder
Connections:
- net C0: now also U2.18 (PB4); no longer U2.9 (PD3)
- net C1: now also U2.20 (PB6); no longer U2.23 (PC6)
- net C2: now also U2.22 (PC7); no longer U2.21 (PB7)
- net C3: now also U2.13 (~{HWB}/PD7); no longer U2.20 (PB6)
- net LED_DATA: now also U2.25 (PC5); no longer U2.15 (PB1)
- net R0: now also U2.7 (PD1); no longer U2.14 (PB0)
- net R1: now also U2.23 (PC6); no longer U2.16 (PB2)
- net R2: now also U2.19 (PB5); no longer U2.25 (PC5)
- net R3: now also U2.21 (PB7); no longer U2.22 (PC7)
- net R4: now also U2.12 (PD6); no longer U2.11 (PD5)
- net R5: now also U2.17 (PB3); no longer U2.10 (PD4)
- net at C3.1, Y1.3: now also U2.1 (XTAL1); no longer U2.2 (PC0/XTAL2)
- net at C1.2, Y1.1: now also U2.2 (PC0/XTAL2); no longer U2.1 (XTAL1)
- no-connect marks 1 -> 13
Other:
- moved on the sheet: R2, R3
Changed lines of the file:
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@@
 	(title_block
 		(title "KiPad")
-		(date "2024-07-23")
-		(rev "3.0")
+		(date "2024-07-30")
+		(rev "3.1")
 		(company "Mechanical & Electrical Industry Research Labs")
 		(comment 1 "Brian Hong")
@@
 	)
 	(junction
+		(at 234.95 162.56)
+		(diameter 0)
+		(color 0 0 0 0)
+	)
+	(junction
 		(at 138.43 85.09)
 		(diameter 0)
@@
 	)
 	(junction
+		(at 212.09 39.37)
+		(diameter 0)
+		(color 0 0 0 0)
+	)
+	(junction
 		(at 33.02 54.61)
 		(diameter 0)
@@
 	)
 	(junction
-		(at 228.6 162.56)
-		(diameter 0)
-		(color 0 0 0 0)
-	)
-	(junction
 		(at 153.67 105.41)
 		(diameter 0)
@@
 	)
 	(junction
-		(at 212.09 39.37)
-		(diameter 0)
-		(color 0 0 0 0)
-	)
-	(junction
 		(at 153.67 39.37)
 		(diameter 0)
@@
 	)
 	(no_connect
+		(at 247.65 36.83)
+	)
+	(no_connect
+		(at 247.65 77.47)
+	)
+	(no_connect
+		(at 229.87 152.4)
+	)
+	(no_connect
+		(at 247.65 82.55)
+	)
+	(no_connect
+		(at 247.65 85.09)
+	)
+	(no_connect
+		(at 247.65 39.37)
+	)
+	(no_connect
+		(at 247.65 34.29)
+	)
+	(no_connect
+		(at 247.65 80.01)
+	)
+	(no_connect
+		(at 247.65 59.69)
+	)
+	(no_connect
+		(at 247.65 72.39)
+	)
+	(no_connect
 		(at 161.29 133.35)
 	)
+	(no_connect
+		(at 229.87 154.94)
+	)
+	(no_connect
+		(at 247.65 57.15)
+	)
 	(wire
 		(pts
@@
 	(wire
 		(pts
-			(xy 231.14 146.05) (xy 231.14 132.08)
+			(xy 231.14 148.59) (xy 231.14 132.08)
 		)
 		(stroke
@@
 	(wire
 		(pts
-			(xy 228.6 158.75) (xy 228.6 162.56)
+			(xy 234.95 158.75) (xy 234.95 162.56)
 		)
 		(stroke
@@
 	(wire
 		(pts
-			(xy 191.77 44.45) (xy 204.47 44.45)
+			(xy 191.77 44.45) (xy 212.09 44.45)
 		)
 		(stroke
@@
 	(wire
 		(pts
-			(xy 232.41 147.32) (xy 231.14 147.32)
+			(xy 237.49 147.32) (xy 232.41 147.32)
 		)
 		(stroke
@@
 	(wire
 		(pts
-			(xy 207.01 44.45) (xy 212.09 44.45)
-		)
-		(stroke
-			(width 0)
-			(type default)
-		)
-	)
-	(wire
-		(pts
-			(xy 231.14 147.32) (xy 231.14 151.13)
+			(xy 237.49 147.32) (xy 237.49 151.13)
 		)
 		(stroke
@@
 	(wire
 		(pts
-			(xy 228.6 162.56) (xy 214.63 162.56)
+			(xy 214.63 162.56) (xy 234.95 162.56)
 		)
 		(stroke
@@
 	(wire
 		(pts
-			(xy 207.01 30.48) (xy 207.01 44.45)
-		)
-		(stroke
-			(width 0)
-			(type default)
-		)
-	)
-	(wire
-		(pts
 			(xy 113.03 59.69) (xy 113.03 80.01)
 		)
@@
 	(wire
 		(pts
-			(xy 228.6 151.13) (xy 228.6 146.05)
+			(xy 234.95 151.13) (xy 234.95 148.59)
 		)
 		(stroke
@@
 	(wire
 		(pts
-			(xy 231.14 158.75) (xy 231.14 162.56)
+			(xy 237.49 158.75) (xy 237.49 162.56)
 		)
 		(stroke
@@
 	(wire
 		(pts
-			(xy 231.14 162.56) (xy 228.6 162.56)
+			(xy 237.49 162.56) (xy 234.95 162.56)
 		)
 		(stroke
@@
 	(wire
 		(pts
+			(xy 208.28 39.37) (xy 212.09 39.37)
+		)
+		(stroke
+			(width 0)
+			(type default)
+		)
+	)
+	(wire
+		(pts
 			(xy 113.03 39.37) (xy 113.03 59.69)
 		)
@@
 	(wire
 		(pts
+			(xy 208.28 30.48) (xy 208.28 39.37)
+		)
+		(stroke
+			(width 0)
+			(type default)
+		)
+	)
+	(wire
+		(pts
 			(xy 83.82 62.23) (xy 102.87 62.23)
 		)
@@
 	(wire
 		(pts
-			(xy 204.47 44.45) (xy 204.47 39.37)
-		)
-		(stroke
-			(width 0)
-			(type default)
-		)
-	)
-	(wire
-		(pts
 			(xy 153.67 80.01) (xy 138.43 80.01)
 		)
@@
 	(wire
 		(pts
-			(xy 228.6 146.05) (xy 231.14 146.05)
+			(xy 234.95 148.59) (xy 231.14 148.59)
 		)
 		(stroke
@@
 	(wire
 		(pts
-			(xy 207.01 30.48) (xy 204.47 30.48)
+			(xy 208.28 30.48) (xy 204.47 30.48)
 		)
 		(stroke
@@
 	(wire
 		(pts
-			(xy 204.47 39.37) (xy 212.09 39.37)
-		)
-		(stroke
-			(width 0)
-			(type default)
-		)
-	)
-	(wire
-		(pts
 			(xy 153.67 24.13) (xy 168.91 24.13)
 		)
@@
 	)
 	(label "C2"
-		(at 247.65 52.07 0)
+		(at 247.65 67.31 0)
 		(fields_autoplaced yes)
 		(effects
@@
 	)
 	(label "R4"
-		(at 247.65 85.09 0)
+		(at 247.65 87.63 0)
 		(fields_autoplaced yes)
 		(effects
@@
 	)
 	(label "R5"
-		(at 247.65 82.55 0)
+		(at 247.65 41.91 0)
 		(fields_autoplaced yes)
 		(effects
@@
 	)
 	(label "R1"
-		(at 247.65 39.37 0)
+		(at 247.65 64.77 0)
 		(fields_autoplaced yes)
 		(effects
@@
 	)
 	(label "C3"
-		(at 247.65 49.53 0)
+		(at 247.65 90.17 0)
 		(fields_autoplaced yes)
 		(effects
@@
 	)
 	(label "LED_DATA"
-		(at 247.65 36.83 0)
+		(at 247.65 62.23 0)
 		(fields_autoplaced yes)
 		(effects
@@
 	)
 	(label "R0"
-		(at 247.65 34.29 0)
+		(at 247.65 74.93 0)
 		(fields_autoplaced yes)
 		(effects
@@
 	)
 	(label "C0"
-		(at 247.65 80.01 0)
+		(at 247.65 44.45 0)
 		(fields_autoplaced yes)
 		(effects
@@
 	)
 	(label "R3"
-		(at 247.65 67.31 0)
+		(at 247.65 52.07 0)
 		(fields_autoplaced yes)
 		(effects
@@
 	)
 	(label "R2"
-		(at 247.65 62.23 0)
+		(at 247.65 46.99 0)
 		(fields_autoplaced yes)
 		(effects
@@
 	)
 	(label "C1"
-		(at 247.65 64.77 0)
+		(at 247.65 49.53 0)
 		(fields_autoplaced yes)
 		(effects
@@
 			)
 		)
-		(property "Footprint" "MX_Hotswap:MX-Hotswap-2U-Vertical-ReversedStabilizers"
+		(property "Footprint" "MX_Hotswap:MX-Hotswap-2U-Vertical"
 			(at 88.9 71.12 0)
 			(effects
@@
 			)
 		)
-		(property "Footprint" "MX_Hotswap:MX-Hotswap-2U"
+		(property "Footprint" "MX_Hotswap:MX-Hotswap-2U-ReversedStabilizers"
 			(at 27.94 120.65 0)
 			(effects
@@
 	)
 	(symbol
-		(lib_id "Connector:USB_C_Receptacle_USB2.0_14P")
+		(lib_id "Connector:USB_C_Receptacle_USB2.0_16P")
 		(at 214.63 139.7 0)
 		(unit 1)
@@
 			)
 		)
-		(property "Description" "USB 2.0-only 14P Type-C Receptacle connector"
+		(property "Description" "USB 2.0-only 16P Type-C Receptacle connector"
 			(at 214.63 139.7 0)
 			(effects
@@
 		(pin "A5"
 		)
+		(pin "A8"
+		)
+		(pin "B8"
+		)
 		(instances
 			(project ""
@@
 			)
 		)
-		(property "Footprint" "MX_Hotswap:MX-Hotswap-2U-Vertical-ReversedStabilizers"
+		(property "Footprint" "MX_Hotswap:MX-Hotswap-2U-Vertical"
 			(at 88.9 104.14 0)
 			(effects
@@
 			)
 		)
-		(property "Footprint" "Resistor_SMD:R_0603_1608Metric"
+		(property "Footprint" "Resistor_SMD:R_0402_1005Metric_Pad0.72x0.64mm_HandSolder"
 			(at 218.44 13.97 0)
 			(effects
@@
 	(symbol
 		(lib_id "Device:R")
-		(at 228.6 154.94 0)
+		(at 234.95 154.94 0)
 		(unit 1)
 		(exclude_from_sim no)
@@
 		(dnp no)
 		(property "Reference" "R2"
-			(at 225.298 150.876 0)
+			(at 231.648 150.876 0)
 			(effects
 				(font
@@
 		)
 		(property "Value" "5.1k"
-			(at 228.6 156.972 90)
+			(at 234.95 156.972 90)
 			(effects
 				(font
@@
 		)
 		(property "Footprint" "Resistor_SMD:R_0402_1005Metric"
-			(at 226.822 154.94 90)
+			(at 233.172 154.94 90)
 			(effects
 				(font
@@
 		)
 		(property "Datasheet" "~"
-			(at 228.6 154.94 0)
+			(at 234.95 154.94 0)
 			(effects
 				(font
@@
 		)
 		(property "Description" "Resistor"
-			(at 228.6 154.94 0)
+			(at 234.95 154.94 0)
 			(effects
 				(font
@@
 		)
 		(property "DIGIKEY" "P5.1KJCT-ND"
-			(at 228.6 154.94 0)
+			(at 234.95 154.94 0)
 			(effects
 				(font
@@
 	(symbol
 		(lib_id "Device:R")
-		(at 231.14 154.94 0)
+		(at 237.49 154.94 0)
 		(mirror y)
 		(unit 1)
@@
 		(dnp no)
 		(property "Reference" "R3"
-			(at 234.442 150.876 0)
+			(at 240.792 150.876 0)
 			(effects
 				(font
@@
 		)
 		(property "Value" "5.1k"
-			(at 231.14 156.972 90)
+			(at 237.49 156.972 90)
 			(effects
 				(font
@@
 		)
 		(property "Footprint" "Resistor_SMD:R_0402_1005Metric"
-			(at 232.918 154.94 90)
+			(at 239.268 154.94 90)
 			(effects
 				(font
@@
 		)
 		(property "Datasheet" "~"
-			(at 231.14 154.94 0)
+			(at 237.49 154.94 0)
 			(effects
 				(font
@@
 		)
 		(property "Description" "Resistor"
-			(at 231.14 154.94 0)
+			(at 237.49 154.94 0)
 			(effects
 				(font
@@
 		)
 		(property "DIGIKEY" "P5.1KJCT-ND"
-			(at 231.14 154.94 0)
+			(at 237.49 154.94 0)
 			(effects
 				(font
